File: altimetro.kicad_sch (KiCad schematic)
At the start: 54 parts, among them J1 BAT 4-16 V, J2 SWD, J3 USB micro-B, J4 PIRO APOGEU, J5 PIRO PRINCIPAL, Q1 AO3400A, Q2 AO3400A, Q3 BSS138, U1 MCP1703A-3302E/MB, U2 STM32F042K6T6, U3 MS5607-02BA03, U4 W25Q16JVSSIQ, U5 USBLC6-2SC6

Commit message: feat: initial commit
Parts:
- J1, J4, J5: footprint TerminalBlock:TerminalBlock_bornier-2_P5.08mm -> TerminalBlock_Phoenix:TerminalBlock_Phoenix_MKDS-1,5-2-5.08_1x02_P5.08mm_Horizontal; symbol Connector_Generic:Conn_01x02 -> Connector:Screw_Terminal_01x02
- U4: footprint Package_SO:SOIC-8_5.23x5.23mm_P1.27mm -> Package_SO:SOIC-8_5.3x5.3mm_P1.27mm
Connections:
- net GND: now also J3.SH (Shield), U1.1 (GND); no longer J3.6 (Shield), U1.2 (VI)
- net VSYS: now also U1.2 (VI); no longer U1.1 (GND)
Other:
- moved on the sheet: C1, C10, C11, C16, C17, C2, C3, C4, C5, C6, C7, C8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

Commit message: feat: PCB feita
Parts:
- J1, J4, J5: footprint TerminalBlock_Phoenix:TerminalBlock_Phoenix_MKDS-1,5-2-5.08_1x02_P5.08mm_Horizontal -> TerminalBlock_MetzConnect:TerminalBlock_MetzConnect_Type059_RT06302HBWC_1x02_P3.50mm_Horizontal
- JP1: now left out of the parts list
Changed lines of the file:
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@@
 			)
 		)
-		(property "Footprint" "TerminalBlock_Phoenix:TerminalBlock_Phoenix_MKDS-1,5-2-5.08_1x02_P5.08mm_Horizontal"
+		(property "Footprint" "TerminalBlock_MetzConnect:TerminalBlock_MetzConnect_Type059_RT06302HBWC_1x02_P3.50mm_Horizontal"
 			(at 40.64 45.72 0)
 			(hide yes)
@@
 		(body_style 1)
 		(exclude_from_sim no)
-		(in_bom yes)
+		(in_bom no)
 		(on_board yes)
 		(in_pos_files yes)
@@
 			)
 		)
-		(property "Footprint" "TerminalBlock_Phoenix:TerminalBlock_Phoenix_MKDS-1,5-2-5.08_1x02_P5.08mm_Horizontal"
+		(property "Footprint" "TerminalBlock_MetzConnect:TerminalBlock_MetzConnect_Type059_RT06302HBWC_1x02_P3.50mm_Horizontal"
 			(at 40.64 167.64 0)
 			(hide yes)
@@
 			)
 		)
-		(property "Footprint" "TerminalBlock_Phoenix:TerminalBlock_Phoenix_MKDS-1,5-2-5.08_1x02_P5.08mm_Horizontal"
+		(property "Footprint" "TerminalBlock_MetzConnect:TerminalBlock_MetzConnect_Type059_RT06302HBWC_1x02_P3.50mm_Horizontal"
 			(at 40.64 256.54 0)
 			(hide yes)
